File: LutrarmyMic_PreAmp/LutrarmyMic_PreAmp.kicad_pcb (KiCad board)
At the start: 2 copper layers, 80 x 80 mm, 56 parts, among them J1 XLR3, J2 XLR3, J3 Conn_01x02_Male, SW1 SW_DPDT_x2, U1 OPA1642, U2 OPA1642

Commit message: 更新最終版 gbr
Parts:
- removed C19: 0.1uF, Capacitor_THT:C_Rect_L7.2mm_W2.5mm_P5.00mm_FKS2_FKP2_MKS2_MKP2
- removed J3: Conn_01x02_Male, Connector_PinHeader_2.54mm:PinHeader_1x02_P2.54mm_Vertical
- removed REF** (x4): MountingHole_3.2mm_M3_ISO7380_Pad, MountingHole:MountingHole_3.2mm_M3_ISO7380_Pad
- removed SW1: SW_DPDT_x2, Connector_PinHeader_2.54mm:PinHeader_1x06_P2.54mm_Vertical
- added H1: MountingHole_Pad, MountingHole:MountingHole_3.2mm_M3_DIN965_Pad, F.Cu at (131.0, 65.9)
- added H2: MountingHole_Pad, MountingHole:MountingHole_3.2mm_M3_DIN965_Pad, F.Cu at (131.0, 133.9)
- added H3: MountingHole_Pad, MountingHole:MountingHole_3.2mm_M3_DIN965_Pad, F.Cu at (199.0, 65.9)
- added H4: MountingHole_Pad, MountingHole:MountingHole_3.2mm_M3_DIN965_Pad, F.Cu at (199.0, 133.9)
- R3, R4: value 1G -> 10M
- moved C2 12.9 mm to (147.0, 89.0), turned to 90 degrees
- moved C14 11.7 mm to (152.0, 122.4), turned to -90 degrees
- moved C13 11.6 mm to (178.0, 122.5), turned to -90 degrees
- moved R21 3.50 mm to (191.0, 118.8)
- moved R23 2.75 mm to (139.5, 118.8)
- moved LutrarmyMic 1.01 mm to (201.3, 120.0)
- turned C11 to -90 degrees
- turned C12 to -90 degrees
Connections:
- C11 pad 1: Net-(C11-Pad1) -> XLR1_48V
- C12 pad 1: Net-(C12-Pad1) -> XLR2_48V
- C13 pad 1: Net-(C11-Pad1) -> XLR1_48V
- C14 pad 1: Net-(C12-Pad1) -> XLR2_48V
- D1 pad 1: Net-(C11-Pad1) -> XLR1_48V
- D2 pad 1: Net-(C12-Pad1) -> XLR2_48V
- R13 pad 1: Net-(C11-Pad1) -> XLR1_48V
- R14 pad 1: Net-(C12-Pad1) -> XLR2_48V
- R15 pad 2: Net-(C11-Pad1) -> XLR1_48V
- R16 pad 2: Net-(C12-Pad1) -> XLR2_48V
Routing:
- net Net-(C12-Pad1): track 59.5 -> 0.00 mm
- net Net-(C11-Pad1): track 59.5 -> 0.00 mm
- net BAT_48V: track 32.5 -> 0.00 mm
- net XLR1_48V: track 45.1 -> 74.7 mm
- net XLR2_48V: track 51.9 -> 74.6 mm
- net Net-(C10-Pad1): track 74.2 -> 62.1 mm
- net Net-(C1-Pad1): track 71.9 -> 64.1 mm
- net Net-(J1-Pad2): track 8.43 -> 11.9 mm
- net Net-(C3-Pad1): track 16.6 -> 13.1 mm
- net Net-(J2-Pad2): track 8.53 -> 11.3 mm
- net Net-(C5-Pad1): track 16.5 -> 13.8 mm
- net Net-(MK1-Pad2): track 36.8 -> 34.3 mm
- net Net-(C6-Pad2): track 18.6 -> 17.9 mm
Other:
- board text added: "Mic1"
- board text added: "Mic1_OUT"
- board text added: "Mic2"
- board text added: "Mic2_OUT"
- board text added: "MicPreAMP V1.1"
- board text removed: "MicPreAMP V1.0"
