File: LutrarmyMic_PreAmp/LutrarmyMic_PreAmp.kicad_sch (KiCad schematic)
At the start: 55 parts, among them J1 XLR3, J2 XLR3, J3 Conn_01x02_Male, SW1 SW_DPDT_x2, U1 OPA1642, U2 OPA1642

Commit message: 更新最終版 gbr
Parts:
- removed C19: 0.1uF, Capacitor_THT:C_Rect_L7.2mm_W2.5mm_P5.00mm_FKS2_FKP2_MKS2_MKP2, symbol Device:C
- removed J3: Conn_01x02_Male, Connector_PinHeader_2.54mm:PinHeader_1x02_P2.54mm_Vertical, symbol Connector:Conn_01x02_Male
- removed SW1: SW_DPDT_x2, symbol Switch:SW_DPDT_x2
- added H1, H2, H3, H4: MountingHole_Pad, MountingHole:MountingHole_3.2mm_M3_DIN965_Pad, symbol Mechanical:MountingHole_Pad
- R15, R16: value 324K -> 21K
- R3, R4: value 1G -> 10M
Connections:
- net Earth: now also H1.1, H2.1, H3.1, H4.1
- net XLR1_48V: now also C11.1, C13.1, D1.1 (K), R13.1, R15.2
- net XLR2_48V: now also C12.1, C14.1, D2.1 (K), R14.1, R16.2
